File: hardware/kicad/LED_MODE.kicad_sch (KiCad schematic)
At the start: 2 parts

Commit message: KiCad v0.2: pinout ESP32 DevKit 30 pines, botones con pull-up interna, buzzer a 5 V, resistencias SMD, logo
Parts:
- D3: footprint LED_THT:LED_D5.0mm -> Connector_Molex:Molex_KK-254_AE-6410-02A_1x02_P2.54mm_Vertical
- R18: footprint Resistor_THT:R_Axial_DIN0207_L6.3mm_D2.5mm_P10.16mm_Horizontal -> Resistor_SMD:R_0805_2012Metric
Changed lines of the file:
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@@
 			)
 		)
-		(property "Footprint" "Resistor_THT:R_Axial_DIN0207_L6.3mm_D2.5mm_P10.16mm_Horizontal"
+		(property "Footprint" "Resistor_SMD:R_0805_2012Metric"
 			(at 144.272 87.63 90)
 			(effects
@@
 			)
 		)
-		(property "Footprint" "LED_THT:LED_D5.0mm"
+		(property "Footprint" "Connector_Molex:Molex_KK-254_AE-6410-02A_1x02_P2.54mm_Vertical"
 			(at 146.05 101.6 0)
 			(effects
