File: hardware/kicad/RAPIDITO [tiempo-reacción].kicad_sch (KiCad schematic)
At the start: 28 parts, among them J2 Screw_Terminal_01x19, J3 Screw_Terminal_01x19, Q1 2N3904

Commit message: KiCad v0.2: pinout ESP32 DevKit 30 pines, botones con pull-up interna, buzzer a 5 V, resistencias SMD, logo
Parts:
- removed J2, J3: Screw_Terminal_01x19, Connector_PinHeader_2.54mm:PinHeader_1x19_P2.54mm_Vertical, symbol Connector:Screw_Terminal_01x19
- removed R12, R14, R4, R8: 10kΩ, Resistor_THT:R_Axial_DIN0207_L6.3mm_D2.5mm_P10.16mm_Horizontal, symbol Device:R
- added J1, J2: Screw_Terminal_01x15, Connector_PinHeader_2.54mm:PinHeader_1x15_P2.54mm_Vertical, symbol Connector:Screw_Terminal_01x15
- BAR1: footprint Connector_PinHeader_1.00mm:PinHeader_1x10_P1.00mm_Vertical -> Connector_PinHeader_2.54mm:PinHeader_1x10_P2.54mm_Vertical
- BTN_MODE1, BTN_RESET1, BTN_RESP1, BTN_START1: footprint Button_Switch_THT:SW_PUSH_6mm -> Connector_Molex:Molex_KK-254_AE-6410-02A_1x02_P2.54mm_Vertical
- D1: footprint Diode_THT:D_DO-41_SOD81_P10.16mm_Horizontal -> Diode_SMD:D_SOD-123
- D2: footprint LED_THT:LED_D5.0mm -> Connector_Molex:Molex_KK-254_AE-6410-02A_1x02_P2.54mm_Vertical
- R1, R2, R3: footprint Resistor_THT:R_Axial_DIN0207_L6.3mm_D2.5mm_P10.16mm_Horizontal -> Resistor_SMD:R_0805_2012Metric
- R10: renamed from R13; footprint Resistor_THT:R_Axial_DIN0207_L6.3mm_D2.5mm_P10.16mm_Horizontal -> Resistor_SMD:R_0805_2012Metric
- R11: renamed from R15; footprint Resistor_THT:R_Axial_DIN0207_L6.3mm_D2.5mm_P10.16mm_Horizontal -> Resistor_SMD:R_0805_2012Metric
- R12: renamed from R16; footprint Resistor_THT:R_Axial_DIN0207_L6.3mm_D2.5mm_P10.16mm_Horizontal -> Resistor_SMD:R_0805_2012Metric
- R13: renamed from R17; footprint Resistor_THT:R_Axial_DIN0207_L6.3mm_D2.5mm_P10.16mm_Horizontal -> Resistor_SMD:R_0805_2012Metric
- R4: renamed from R5; footprint Resistor_THT:R_Axial_DIN0207_L6.3mm_D2.5mm_P10.16mm_Horizontal -> Resistor_SMD:R_0805_2012Metric
- R5: renamed from R6; footprint Resistor_THT:R_Axial_DIN0207_L6.3mm_D2.5mm_P10.16mm_Horizontal -> Resistor_SMD:R_0805_2012Metric
- R6: renamed from R7; footprint Resistor_THT:R_Axial_DIN0207_L6.3mm_D2.5mm_P10.16mm_Horizontal -> Resistor_SMD:R_0805_2012Metric
- R7: renamed from R9; footprint Resistor_THT:R_Axial_DIN0207_L6.3mm_D2.5mm_P10.16mm_Horizontal -> Resistor_SMD:R_0805_2012Metric
- R8: renamed from R10; footprint Resistor_THT:R_Axial_DIN0207_L6.3mm_D2.5mm_P10.16mm_Horizontal -> Resistor_SMD:R_0805_2012Metric
- R9: renamed from R11; footprint Resistor_THT:R_Axial_DIN0207_L6.3mm_D2.5mm_P10.16mm_Horizontal -> Resistor_SMD:R_0805_2012Metric
Connections:
- net BUZZER: now also J2.6 (Pin_6)
- net GND: now also J1.2 (Pin_2), J2.2 (Pin_2)
- net LED1: now also J1.15 (Pin_15)
- net LED10: now also J2.3 (Pin_3)
- net LED2: now also J1.14 (Pin_14)
- net LED3: now also J1.11 (Pin_11)
- net LED4: now also J1.10 (Pin_10)
- net LED5: now also J1.9 (Pin_9)
- net LED6: now also J1.7 (Pin_7)
- net LED7: now also J1.6 (Pin_6)
- net LED8: now also J1.5 (Pin_5)
- net LED9: now also J2.5 (Pin_5)
- net LED_MODE: now also J1.8 (Pin_8)
- net MODE_input: now also J2.7 (Pin_7)
- net RESET_input: now also J2.8 (Pin_8)
- net RESP_input: now also J2.10 (Pin_10)
- net START_input: now also J2.9 (Pin_9)
- net VCC_3V3: now also J1.1 (Pin_1); no longer BZ1.1 (+), D1.1 (K)
- net VCC_5V: now also BZ1.1 (+), D1.1 (K), J2.1 (Pin_1)
